File: hardware/Robot Controller.sch (EAGLE design)
At the start: 18 parts, among them U1 ATMEGA328P_PDIP

Commit message: WIP hardware
Parts:
- removed H1: MOUNT-HOLE2.8, holes:MOUNT-HOLE2.8
- JP7: device pinhead:PINHD-2X13 -> pinhead:PINHD-1X4
Connections:
- net DEBUG' renamed DEBUG
- removed net M2PW': L293D.9, R3.2
- new net ADC0: JP7.1, U1.PC0(ADC0)
- new net ADC1: JP7.2, U1.PC1(ADC1)
- new net ADC2: JP7.3, U1.PC2(ADC2)
- new net ADC3: JP7.4, U1.PC3(ADC3)
- new net M2PW: L293D.9, R3.2, U1.PB1(OC1A)
- net 3.3V: now also U1.AVCC
Other:
- note added: "ADC0"
- note added: "ADC1"
- note added: "ADC2"
- note added: "ADC3"
- note added: "DEBUG"
- note added: "M2PW"
- note removed: "DEBUG'"
- note removed: "M2PW'"
Changed lines of the file:
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@@
 <part name="R1" library="resistor" deviceset="R-US_" device="R3216"/>
 <part name="LED1" library="led" deviceset="LED" device="SMT1206"/>
-<part name="H1" library="holes" deviceset="MOUNT-HOLE" device="2.8"/>
 <part name="R3" library="resistor" deviceset="R-US_" device="R3216"/>
 <part name="LED3" library="led" deviceset="LED" device="SMT1206"/>
@@
 <part name="GND11" library="SparkFun-Aesthetics" deviceset="GND" device=""/>
 <part name="GND13" library="SparkFun-Aesthetics" deviceset="GND" device=""/>
-<part name="JP7" library="pinhead" deviceset="PINHD-2X13" device=""/>
+<part name="SUPPLY2" library="SparkFun-Aesthetics" deviceset="3.3V" device=""/>
+<part name="JP7" library="pinhead" deviceset="PINHD-1X4" device=""/>
 </parts>
 <sheets>
@@
 <text x="142.24" y="104.14" size="1.778" layer="95" rot="R270">M1PW'</text>
 <text x="-33.02" y="33.02" size="1.778" layer="95">M1PW'</text>
-<text x="157.48" y="99.06" size="1.778" layer="95" rot="R90">M2PW'</text>
-<text x="-7.62" y="12.7" size="1.778" layer="95" rot="R180">M2PW'</text>
+<text x="157.48" y="99.06" size="1.778" layer="95" rot="R90">M2PW</text>
+<text x="-15.24" y="10.16" size="1.778" layer="95">M2PW</text>
 <text x="-33.02" y="15.24" size="1.778" layer="95" rot="R180">M1DR'</text>
 <text x="-12.7" y="73.66" size="1.778" layer="95" rot="R180">M1DR'</text>
@@
 <text x="-20.32" y="63.5" size="1.778" layer="95">M2DR_'</text>
 <text x="-15.24" y="25.4" size="1.778" layer="95">M2DR_'</text>
-<text x="43.18" y="83.82" size="1.778" layer="95" rot="R90">DEBUG'</text>
+<text x="43.18" y="83.82" size="1.778" layer="95" rot="R90">DEBUG</text>
 <text x="68.58" y="81.28" size="1.778" layer="95" rot="R90">HOST'</text>
 <text x="27.94" y="38.1" size="1.778" layer="95">RESET'</text>
 <text x="96.52" y="83.82" size="1.778" layer="95" rot="R90">SS'</text>
-<text x="88.9" y="-10.16" size="1.778" layer="95" rot="R180">SS'</text>
+<text x="86.36" y="-12.7" size="1.778" layer="95">SS'</text>
 <text x="83.82" y="-17.78" size="1.778" layer="95">MISO'</text>
 <text x="83.82" y="-15.24" size="1.778" layer="95">MOSI'</text>
 <text x="83.82" y="-20.32" size="1.778" layer="95">SCL'</text>
 <text x="83.82" y="0" size="1.778" layer="95">M1PW'</text>
-<text x="83.82" y="15.24" size="1.778" layer="95">DEBUG'</text>
+<text x="83.82" y="15.24" size="1.778" layer="95">DEBUG</text>
 <text x="83.82" y="12.7" size="1.778" layer="95">HOST'</text>
 <text x="83.82" y="10.16" size="1.778" layer="95">M1DR'</text>
 <text x="83.82" y="7.62" size="1.778" layer="95">M2DR'</text>
+<text x="83.82" y="-10.16" size="1.778" layer="95">M2PW</text>
+<text x="86.36" y="38.1" size="1.778" layer="95">ADC0</text>
+<text x="101.6" y="40.64" size="1.778" layer="95">ADC0</text>
+<text x="86.36" y="35.56" size="1.778" layer="95">ADC1</text>
+<text x="101.6" y="38.1" size="1.778" layer="95">ADC1</text>
+<text x="101.6" y="35.56" size="1.778" layer="95">ADC2</text>
+<text x="86.36" y="33.02" size="1.778" layer="95">ADC2</text>
+<text x="86.36" y="30.48" size="1.778" layer="95">ADC3</text>
+<text x="101.6" y="33.02" size="1.778" layer="95">ADC3</text>
 </plain>
 <instances>
@@
 <instance part="R1" gate="G$1" x="144.78" y="93.98" rot="R90"/>
 <instance part="LED1" gate="G$1" x="144.78" y="83.82"/>
-<instance part="H1" gate="G$1" x="-35.56" y="114.3"/>
 <instance part="R3" gate="G$1" x="157.48" y="93.98" rot="R90"/>
 <instance part="LED3" gate="G$1" x="157.48" y="83.82"/>
@@
 <instance part="GND11" gate="1" x="25.4" y="-15.24" rot="R270"/>
 <instance part="GND13" gate="1" x="27.94" y="-20.32"/>
-<instance part="JP7" gate="A" x="127" y="114.3" rot="R90"/>
+<instance part="SUPPLY2" gate="G$1" x="27.94" y="33.02" rot="R90"/>
+<instance part="JP7" gate="A" x="116.84" y="35.56"/>
 </instances>
 <busses>
@@
 <pinref part="SUPPLY8" gate="G$1" pin="3.3V"/>
 </segment>
+<segment>
+<pinref part="U1" gate="G$1" pin="AVCC"/>
+<wire x1="33.02" y1="33.02" x2="27.94" y2="33.02" width="0.1524" layer="91"/>
+<pinref part="SUPPLY2" gate="G$1" pin="3.3V"/>
+</segment>
 </net>
 <net name="5V" class="0">
@@
 </segment>
 </net>
-<net name="M2PW'" class="0">
-<segment>
-<pinref part="R3" gate="G$1" pin="2"/>
-<wire x1="157.48" y1="99.06" x2="157.48" y2="104.14" width="0.1524" layer="91"/>
-</segment>
-<segment>
-<pinref part="L293D" gate="G$1" pin="9"/>
-<wire x1="-10.16" y1="10.16" x2="-17.78" y2="10.16" width="0.1524" layer="91"/>
-<junction x="-17.78" y="10.16"/>
-</segment>
-</net>
 <net name="M1DR'" class="0">
 <segment>
@@
 <pinref part="U1" gate="G$1" pin="PD3(INT1)"/>
 <wire x1="81.28" y1="7.62" x2="88.9" y2="7.62" width="0.1524" layer="91"/>
-</segment>
-</net>
-<net name="DEBUG'" class="0">
-<segment>
-<wire x1="43.18" y1="83.82" x2="43.18" y2="88.9" width="0.1524" layer="91"/>
-<wire x1="43.18" y1="88.9" x2="43.18" y2="91.44" width="0.1524" layer="91"/>
-<pinref part="JP6" gate="A" pin="2"/>
-<wire x1="43.18" y1="91.44" x2="35.56" y2="91.44" width="0.1524" layer="91"/>
-<junction x="35.56" y="91.44"/>
-</segment>
-<segment>
-<pinref part="U1" gate="G$1" pin="PD0(RXD)"/>
-<wire x1="81.28" y1="15.24" x2="88.9" y2="15.24" width="0.1524" layer="91"/>
 </segment>
 </net>
@@
 </segment>
 </net>
+<net name="M2PW" class="0">
+<segment>
+<pinref part="U1" gate="G$1" pin="PB1(OC1A)"/>
+<wire x1="81.28" y1="-10.16" x2="88.9" y2="-10.16" width="0.1524" layer="91"/>
+</segment>
+<segment>
+<pinref part="L293D" gate="G$1" pin="9"/>
+<wire x1="-7.62" y1="10.16" x2="-17.78" y2="10.16" width="0.1524" layer="91"/>
+<junction x="-17.78" y="10.16"/>
+</segment>
+<segment>
+<pinref part="R3" gate="G$1" pin="2"/>
+<wire x1="157.48" y1="99.06" x2="157.48" y2="104.14" width="0.1524" layer="91"/>
+</segment>
+</net>
+<net name="ADC0" class="0">
+<segment>
+<pinref part="JP7" gate="A" pin="1"/>
+<wire x1="114.3" y1="40.64" x2="104.14" y2="40.64" width="0.1524" layer="91"/>
+</segment>
+<segment>
+<pinref part="U1" gate="G$1" pin="PC0(ADC0)"/>
+<wire x1="81.28" y1="38.1" x2="91.44" y2="38.1" width="0.1524" layer="91"/>
+</segment>
+</net>
+<net name="ADC1" class="0">
+<segment>
+<pinref part="JP7" gate="A" pin="2"/>
+<wire x1="114.3" y1="38.1" x2="101.6" y2="38.1" width="0.1524" layer="91"/>
+</segment>
+<segment>
+<pinref part="U1" gate="G$1" pin="PC1(ADC1)"/>
+<wire x1="81.28" y1="35.56" x2="91.44" y2="35.56" width="0.1524" layer="91"/>
+</segment>
+</net>
+<net name="ADC2" class="0">
+<segment>
+<pinref part="JP7" gate="A" pin="3"/>
+<wire x1="114.3" y1="35.56" x2="101.6" y2="35.56" width="0.1524" layer="91"/>
+</segment>
+<segment>
+<pinref part="U1" gate="G$1" pin="PC2(ADC2)"/>
+<wire x1="81.28" y1="33.02" x2="91.44" y2="33.02" width="0.1524" layer="91"/>
+</segment>
+</net>
+<net name="ADC3" class="0">
+<segment>
+<pinref part="JP7" gate="A" pin="4"/>
+<wire x1="114.3" y1="33.02" x2="101.6" y2="33.02" width="0.1524" layer="91"/>
+</segment>
+<segment>
+<pinref part="U1" gate="G$1" pin="PC3(ADC3)"/>
+<wire x1="81.28" y1="30.48" x2="91.44" y2="30.48" width="0.1524" layer="91"/>
+</segment>
+</net>
+<net name="DEBUG" class="0">
+<segment>
+<pinref part="U1" gate="G$1" pin="PD0(RXD)"/>
+<wire x1="81.28" y1="15.24" x2="88.9" y2="15.24" width="0.1524" layer="91"/>
+</segment>
+<segment>
+<wire x1="43.18" y1="83.82" x2="43.18" y2="88.9" width="0.1524" layer="91"/>
+<wire x1="43.18" y1="88.9" x2="43.18" y2="91.44" width="0.1524" layer="91"/>
+<pinref part="JP6" gate="A" pin="2"/>
+<wire x1="43.18" y1="91.44" x2="35.56" y2="91.44" width="0.1524" layer="91"/>
+<junction x="35.56" y="91.44"/>
+</segment>
+</net>

Commit message: more work on rev0.2 hardware
Parts:
- removed JP7: (no value), pinhead:PINHD-1X4
- JP6: device pinhead:PINHD-1X3 -> pinhead:PINHD-1X6
Connections:
- removed net N$21: JP6.1, R2.1
- removed net N$23: JP6.3
- new net ADC4: JP6.5, U1.PC4(ADC4/SDA)
- new net ADC5: JP6.6, U1.PC5(ADC5/SCL)
- net ADC0: now also JP6.1; no longer JP7.1
- net ADC1: now also JP6.2; no longer JP7.2
- net ADC2: now also JP6.3; no longer JP7.3
- net ADC3: now also JP6.4; no longer JP7.4
- net DEBUG: now also R2.1; no longer JP6.2
Other:
- note added: "ADC4"
- note added: "ADC5"
Changed lines of the file:
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@@
 <part name="JP5" library="pinhead" deviceset="PINHD-1X7" device=""/>
 <part name="GND10" library="SparkFun-Aesthetics" deviceset="GND" device=""/>
-<part name="JP6" library="pinhead" deviceset="PINHD-1X3" device=""/>
 <part name="GND12" library="SparkFun-Aesthetics" deviceset="GND" device=""/>
 <part name="JP8" library="pinhead" deviceset="PINHD-1X2" device=""/>
@@
 <part name="GND13" library="SparkFun-Aesthetics" deviceset="GND" device=""/>
 <part name="SUPPLY2" library="SparkFun-Aesthetics" deviceset="3.3V" device=""/>
-<part name="JP7" library="pinhead" deviceset="PINHD-1X4" device=""/>
+<part name="JP6" library="pinhead" deviceset="PINHD-1X6" device=""/>
 </parts>
 <sheets>
@@
 <text x="-20.32" y="63.5" size="1.778" layer="95">M2DR_'</text>
 <text x="-15.24" y="25.4" size="1.778" layer="95">M2DR_'</text>
-<text x="43.18" y="83.82" size="1.778" layer="95" rot="R90">DEBUG</text>
+<text x="43.18" y="88.9" size="1.778" layer="95" rot="R90">DEBUG</text>
 <text x="68.58" y="81.28" size="1.778" layer="95" rot="R90">HOST'</text>
 <text x="27.94" y="38.1" size="1.778" layer="95">RESET'</text>
@@
 <text x="86.36" y="30.48" size="1.778" layer="95">ADC3</text>
 <text x="101.6" y="33.02" size="1.778" layer="95">ADC3</text>
+<text x="86.36" y="27.94" size="1.778" layer="95">ADC4</text>
+<text x="101.6" y="30.48" size="1.778" layer="95">ADC4</text>
+<text x="86.36" y="25.4" size="1.778" layer="95">ADC5</text>
+<text x="101.6" y="27.94" size="1.778" layer="95">ADC5</text>
 </plain>
 <instances>
@@
 <instance part="JP5" gate="A" x="111.76" y="99.06" rot="R90"/>
 <instance part="GND10" gate="1" x="116.84" y="78.74"/>
-<instance part="JP6" gate="A" x="38.1" y="91.44"/>
 <instance part="GND12" gate="1" x="73.66" y="124.46" rot="R90"/>
 <instance part="JP8" gate="G$1" x="66.04" y="127" rot="R90"/>
@@
 <instance part="GND13" gate="1" x="27.94" y="-20.32"/>
 <instance part="SUPPLY2" gate="G$1" x="27.94" y="33.02" rot="R90"/>
-<instance part="JP7" gate="A" x="116.84" y="35.56"/>
+<instance part="JP6" gate="A" x="116.84" y="33.02"/>
 </instances>
 <busses>
@@
 <wire x1="-7.62" y1="25.4" x2="-17.78" y2="25.4" width="0.1524" layer="91"/>
 <junction x="-17.78" y="25.4"/>
-</segment>
-</net>
-<net name="N$21" class="0">
-<segment>
-<pinref part="JP6" gate="A" pin="1"/>
-<wire x1="35.56" y1="93.98" x2="43.18" y2="93.98" width="0.1524" layer="91"/>
-<pinref part="R2" gate="G$1" pin="1"/>
-<wire x1="43.18" y1="93.98" x2="43.18" y2="99.06" width="0.1524" layer="91"/>
-<junction x="35.56" y="93.98"/>
-<junction x="43.18" y="99.06"/>
-</segment>
-</net>
-<net name="N$23" class="0">
-<segment>
-<pinref part="JP6" gate="A" pin="3"/>
-<wire x1="12.7" y1="88.9" x2="35.56" y2="88.9" width="0.1524" layer="91"/>
-<junction x="35.56" y="88.9"/>
 </segment>
 </net>
@@
 <net name="ADC0" class="0">
 <segment>
-<pinref part="JP7" gate="A" pin="1"/>
 <wire x1="114.3" y1="40.64" x2="104.14" y2="40.64" width="0.1524" layer="91"/>
+<pinref part="JP6" gate="A" pin="1"/>
 </segment>
 <segment>
@@
 <net name="ADC1" class="0">
 <segment>
-<pinref part="JP7" gate="A" pin="2"/>
 <wire x1="114.3" y1="38.1" x2="101.6" y2="38.1" width="0.1524" layer="91"/>
+<pinref part="JP6" gate="A" pin="2"/>
 </segment>
 <segment>
@@
 <net name="ADC2" class="0">
 <segment>
-<pinref part="JP7" gate="A" pin="3"/>
 <wire x1="114.3" y1="35.56" x2="101.6" y2="35.56" width="0.1524" layer="91"/>
+<pinref part="JP6" gate="A" pin="3"/>
 </segment>
 <segment>
@@
 <net name="ADC3" class="0">
 <segment>
-<pinref part="JP7" gate="A" pin="4"/>
 <wire x1="114.3" y1="33.02" x2="101.6" y2="33.02" width="0.1524" layer="91"/>
+<pinref part="JP6" gate="A" pin="4"/>
 </segment>
 <segment>
@@
 </segment>
 <segment>
-<wire x1="43.18" y1="83.82" x2="43.18" y2="88.9" width="0.1524" layer="91"/>
-<wire x1="43.18" y1="88.9" x2="43.18" y2="91.44" width="0.1524" layer="91"/>
-<pinref part="JP6" gate="A" pin="2"/>
-<wire x1="43.18" y1="91.44" x2="35.56" y2="91.44" width="0.1524" layer="91"/>
-<junction x="35.56" y="91.44"/>
-</segment>
-</net>
+<wire x1="43.18" y1="88.9" x2="43.18" y2="93.98" width="0.1524" layer="91"/>
+<pinref part="R2" gate="G$1" pin="1"/>
+<wire x1="43.18" y1="93.98" x2="43.18" y2="99.06" width="0.1524" layer="91"/>
+<junction x="43.18" y="99.06"/>
+</segment>
+</net>
+<net name="ADC4" class="0">
+<segment>
+<pinref part="U1" gate="G$1" pin="PC4(ADC4/SDA)"/>
+<wire x1="81.28" y1="27.94" x2="91.44" y2="27.94" width="0.1524" layer="91"/>
+</segment>
+<segment>
+<pinref part="JP6" gate="A" pin="5"/>
+<wire x1="114.3" y1="30.48" x2="101.6" y2="30.48" width="0.1524" layer="91"/>
+</segment>
+</net>
+<net name="ADC5" class="0">
+<segment>
+<pinref part="U1" gate="G$1" pin="PC5(ADC5/SCL)"/>
+<wire x1="81.28" y1="25.4" x2="91.44" y2="25.4" width="0.1524" layer="91"/>
+</segment>
+<segment>
+<pinref part="JP6" gate="A" pin="6"/>
+<wire x1="114.3" y1="27.94" x2="101.6" y2="27.94" width="0.1524" layer="91"/>
+</segment>
+</net>
